File: KiCAD/DrumPADPCB/DrumPADPCB.kicad_pcb (KiCad board)
At the start: 2 copper layers, 24 parts, among them J1 Conn_01x02_Pin, J3 Conn_01x04_Pin, U1 LM321, U2 LM321

Commit message: Signal Processing Demo PCB almost done
Parts:
- removed TP1, TP2, TP3, TP4, TP5: TestPoint, Connector_Pin:Pin_D1.4mm_L8.5mm_W2.8mm_FlatFork
- added Buffered-Scaled1: TestPoint, Connector_Pin:Pin_D1.4mm_L8.5mm_W2.8mm_FlatFork, F.Cu at (111.2, 81.0)
- added Buffered1: TestPoint, Connector_Pin:Pin_D1.4mm_L8.5mm_W2.8mm_FlatFork, F.Cu at (99.2, 81.0)
- added Filtered1: TestPoint, Connector_Pin:Pin_D1.4mm_L8.5mm_W2.8mm_FlatFork, F.Cu at (86.2, 71.8)
- added RAW1: TestPoint, Connector_Pin:Pin_D1.4mm_L8.5mm_W2.8mm_FlatFork, F.Cu at (77.5, 71.8)
- added Scaled1: TestPoint, Connector_Pin:Pin_D1.4mm_L8.5mm_W2.8mm_FlatFork, F.Cu at (105.2, 81.0)
- J1: footprint Connector_PinHeader_2.54mm:PinHeader_1x02_P2.54mm_Horizontal -> Connector_PinHeader_2.54mm:PinHeader_1x02_P2.54mm_Vertical
- moved J3 99.3 mm to (117.2, 70.5)
- moved C4 96.8 mm to (110.0, 71.0), turned to 180 degrees
- moved C5 96.6 mm to (110.0, 73.5), turned to 180 degrees
- moved C2 88.3 mm to (95.0, 73.5), turned to 180 degrees
- moved D5 87.8 mm to (105.3, 68.5)
- moved D3 87.6 mm to (114.0, 76.8), turned to -90 degrees
- moved C1 86.0 mm to (87.5, 76.0), turned to -90 degrees
- moved U2 85.5 mm to (110.1, 77.0)
- moved C3 85.2 mm to (95.0, 71.0), turned to 180 degrees
- moved D4 79.8 mm to (95.3, 68.5)
- moved R3 76.6 mm to (100.0, 68.5)
- moved U1 76.1 mm to (95.0, 77.0)
- moved R4 75.7 mm to (110.0, 68.5), turned to 180 degrees
- moved R2 74.5 mm to (90.5, 76.0), turned to -90 degrees
- moved R1 67.1 mm to (77.0, 76.5), turned to -90 degrees
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Other:
- board text added: "24V"
- board text added: "3V3"
- board text added: "CCW to increas CW to decrease"
- board text added: "GND"
- board text added: "IN"
- board text added: "OUT"

Commit message: PCB V1.0 release ready to order
Parts:
- added GND1: TestPoint, Connector_Pin:Pin_D1.4mm_L8.5mm_W2.8mm_FlatFork, F.Cu at (84.3, 58.2)
- added GND2: TestPoint, Connector_Pin:Pin_D1.4mm_L8.5mm_W2.8mm_FlatFork, F.Cu at (129.5, 70.1)
- moved Buffered1 17.5 mm to (112.9, 70.0)
- moved Filtered1 17.4 mm to (99.7, 60.8)
- moved J3 17.2 mm to (129.6, 58.4)
- moved J1 16.7 mm to (86.0, 64.0)
- moved U2 16.5 mm to (122.4, 66.0)
- moved Buffered-Scaled1 16.5 mm to (123.5, 70.0)
- moved C1 16.5 mm to (99.8, 65.0)
- moved C2 16.5 mm to (107.3, 62.5)
- moved C3 16.5 mm to (107.3, 60.0)
- moved C4 16.5 mm to (122.3, 60.0)
- moved C5 16.5 mm to (122.3, 62.5)
- moved D1 16.5 mm to (93.0, 64.0)
- moved D2 16.5 mm to (96.8, 65.2)
- moved D3 16.5 mm to (126.3, 65.8)
- moved D5 16.5 mm to (117.6, 57.5)
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Routing:
- net 24V: track 0.00 -> 29.3 mm
- net Net-(D1-K): track 0.00 -> 16.2 mm
- net 3V3: track 0.00 -> 15.4 mm
- net /Piezo Processing Board/Sig_Out: track 0.00 -> 12.8 mm
- net Net-(U1--): track 0.00 -> 10.4 mm
- net Net-(D1-A): track 0.00 -> 10.4 mm
- net Net-(U2-+): track 0.00 -> 9.71 mm
- net Net-(D5-A): track 0.00 -> 2.72 mm
- net Net-(D4-A): track 0.00 -> 2.50 mm
- net GND: vias 0 -> 30
- added copper zone on B.Cu, net GND
- added copper zone on F.Cu, net GND
Other:
- board outline added: 56 x 20 mm
- board text added: "CCW: increas CW : decrease"
- board text added: "PIEZO BOARD by Andy Woo V.1 2024-11-23"
- board text removed: "CCW to increas CW to decrease"
